File: HF/HF.sch (KiCad schematic (older format))
At the start: 13 parts, among them J1 NL4MP-M3, J2 NL4MP-M3, U1 1+, U2 1-, U3 HF-, U4 HF+

Commit message: added everything but the inductor
Parts:
- removed U1: 1+, SpeakON:Reoforo, symbol Reoforo:Reoforo
- removed U2: 1-, SpeakON:Reoforo, symbol Reoforo:Reoforo
- LA1: footprint (none) -> Resistor_THT:R_Axial_Power_L38.0mm_W9.0mm_P45.72mm
Changed lines of the file:
@@
 F 0 "LA1" V 4935 3750 50  0000 C CNN
 F 1 "1,5Ω" V 5026 3750 50  0000 C CNN
-F 2 "" V 5200 3850 50  0001 C CNN
+F 2 "Resistor_THT:R_Axial_Power_L38.0mm_W9.0mm_P45.72mm" V 5200 3850 50  0001 C CNN
 F 3 "~" V 5200 3850 50  0001 C CNN
 	1    5200 3750
@@
 	1    0    0    -1
 $EndComp
-$Comp
-L Reoforo:Reoforo U2
-U 1 1 60A1685A
-P 4150 2700
-F 0 "U2" H 4050 2750 50  0000 L CNN
-F 1 "1-" H 4278 2677 50  0000 L CNN
-F 2 "SpeakON:Reoforo" H 4150 2700 50  0001 C CNN
-F 3 "" H 4150 2700 50  0001 C CNN
-	1    4150 2700
-	1    0    0    -1
-$EndComp
-Wire Wire Line
-	4150 2700 3800 2700
-Connection ~ 3800 2700
-$Comp
-L Reoforo:Reoforo U1
-U 1 1 60A186D9
-P 2600 3750
-F 0 "U1" H 2500 3800 50  0000 L CNN
-F 1 "1+" H 2728 3727 50  0000 L CNN
-F 2 "SpeakON:Reoforo" H 2600 3750 50  0001 C CNN
-F 3 "" H 2600 3750 50  0001 C CNN
-	1    2600 3750
-	-1   0    0    1
-$EndComp
-Wire Wire Line
-	2600 3750 2750 3750
-Connection ~ 2750 3750
 $EndSCHEMATC

Commit message: inductor added
Parts:
- L1: footprint (none) -> RES:inductor_40mm
- R3, R4: footprint Resistor_THT:R_Axial_Power_L25.0mm_W9.0mm_P30.48mm -> RES:resistor_P27.50mm
Changed lines of the file:
@@
 F 0 "R3" V 4993 4150 50  0000 C CNN
 F 1 "3,3Ω" V 5084 4150 50  0000 C CNN
-F 2 "Resistor_THT:R_Axial_Power_L25.0mm_W9.0mm_P30.48mm" V 5130 4150 50  0001 C CNN
+F 2 "RES:resistor_P27.50mm" V 5130 4150 50  0001 C CNN
 F 3 "~" H 5200 4150 50  0001 C CNN
 	1    5200 4150
@@
 F 0 "R4" V 5693 3750 50  0000 C CNN
 F 1 "5,6Ω" V 5784 3750 50  0000 C CNN
-F 2 "Resistor_THT:R_Axial_Power_L25.0mm_W9.0mm_P30.48mm" V 5830 3750 50  0001 C CNN
+F 2 "RES:resistor_P27.50mm" V 5830 3750 50  0001 C CNN
 F 3 "~" H 5900 3750 50  0001 C CNN
 	1    5900 3750
@@
 F 0 "L1" H 6802 4096 50  0000 L CNN
 F 1 "290uH" H 6802 4005 50  0000 L CNN
-F 2 "" H 6750 4050 50  0001 C CNN
+F 2 "RES:inductor_40mm" H 6750 4050 50  0001 C CNN
 F 3 "~" H 6750 4050 50  0001 C CNN
 	1    6750 4050

Commit message: changes from Trello
Parts:
- removed U3: HF-, SpeakON:Reoforo, symbol Reoforo:Reoforo
- removed U4: HF+, SpeakON:Reoforo, symbol Reoforo:Reoforo
- added J3: Conn_01x02_Male, RES:Faston_DUAL_01x02_P5.08mm_D5.08mm, symbol Connector:Conn_01x02_Male
- LA1: footprint Resistor_THT:R_Axial_Power_L38.0mm_W9.0mm_P45.72mm -> RES:lamp
- R1, R2: footprint Fuse:Fuse_Bourns_MF-RHT300 -> RES:ptc_7.2mm_larger
Connections:
- net at C1.1, L1.1: now also J3.2 (Pin_2)
- net at J1.2-, J2.2-, L1.2: now also J3.1 (Pin_1)
Changed lines of the file:
@@
 F 0 "R1" V 4343 3750 50  0000 C CNN
 F 1 "100mΩ" V 4434 3750 50  0000 C CNN
-F 2 "Fuse:Fuse_Bourns_MF-RHT300" V 4480 3750 50  0001 C CNN
+F 2 "RES:ptc_7.2mm_larger" V 4480 3750 50  0001 C CNN
 F 3 "~" H 4550 3750 50  0001 C CNN
 	1    4550 3750
@@
 F 0 "LA1" V 4935 3750 50  0000 C CNN
 F 1 "1,5Ω" V 5026 3750 50  0000 C CNN
-F 2 "Resistor_THT:R_Axial_Power_L38.0mm_W9.0mm_P45.72mm" V 5200 3850 50  0001 C CNN
+F 2 "RES:lamp" V 5200 3850 50  0001 C CNN
 F 3 "~" V 5200 3850 50  0001 C CNN
 	1    5200 3750
@@
 F 0 "R2" V 4343 4150 50  0000 C CNN
 F 1 "100mΩ" V 4434 4150 50  0000 C CNN
-F 2 "Fuse:Fuse_Bourns_MF-RHT300" V 4480 4150 50  0001 C CNN
+F 2 "RES:ptc_7.2mm_larger" V 4480 4150 50  0001 C CNN
 F 3 "~" H 4550 4150 50  0001 C CNN
 	1    4550 4150
@@
 Connection ~ 6750 3750
 Wire Wire Line
-	6750 3750 7150 3750
-Wire Wire Line
 	5050 4150 4850 4150
 Wire Wire Line
@@
 	4100 3750 4250 3750
 Connection ~ 4250 3750
-Wire Wire Line
-	7150 4350 6750 4350
 Connection ~ 6750 4350
 $Comp
@@
 	2750 3050 2800 3050
 $Comp
-L Reoforo:Reoforo U3
-U 1 1 60A16242
-P 7150 3750
-F 0 "U3" H 7050 3800 50  0000 L CNN
-F 1 "HF-" H 7278 3727 50  0000 L CNN
-F 2 "SpeakON:Reoforo" H 7150 3750 50  0001 C CNN
-F 3 "" H 7150 3750 50  0001 C CNN
-	1    7150 3750
-	1    0    0    -1
+L Connector:Conn_01x02_Male J3
+U 1 1 60A4FD2F
+P 7600 4100
+F 0 "J3" H 7572 4074 50  0000 R CNN
+F 1 "Conn_01x02_Male" H 7572 3983 50  0000 R CNN
+F 2 "RES:Faston_DUAL_01x02_P5.08mm_D5.08mm" H 7600 4100 50  0001 C CNN
+F 3 "~" H 7600 4100 50  0001 C CNN
+	1    7600 4100
+	-1   0    0    1
 $EndComp
-$Comp
-L Reoforo:Reoforo U4
-U 1 1 60A1668B
-P 7150 4350
-F 0 "U4" H 7050 4400 50  0000 L CNN
-F 1 "HF+" H 7278 4327 50  0000 L CNN
-F 2 "SpeakON:Reoforo" H 7150 4350 50  0001 C CNN
-F 3 "" H 7150 4350 50  0001 C CNN
-	1    7150 4350
-	1    0    0    -1
-$EndComp
+Wire Wire Line
+	7400 4000 7250 4000
+Wire Wire Line
+	7250 4000 7250 3750
+Wire Wire Line
+	6750 3750 7250 3750
+Wire Wire Line
+	7400 4100 7250 4100
+Wire Wire Line
+	7250 4100 7250 4350
+Wire Wire Line
+	6750 4350 7250 4350
 $EndSCHEMATC

Commit message: added parallel board
Parts:
- J1, J2: footprint SpeakON:NL4MP-M3 -> SpeakON:NL4MP-M3_double_left
Changed lines of the file:
@@
 F 0 "J2" V 3319 3750 50  0000 C CNN
 F 1 "NL4MP-M3" V 3410 3750 50  0000 C CNN
-F 2 "SpeakON:NL4MP-M3" H 3800 3750 50  0001 C CNN
+F 2 "SpeakON:NL4MP-M3_double_left" H 3800 3750 50  0001 C CNN
 F 3 "http://www.neutrik.com/en/speakon/" H 3800 3750 50  0001 C CNN
 	1    3800 3750
@@
 F 0 "J1" V 2619 3050 50  0000 C CNN
 F 1 "NL4MP-M3" V 2710 3050 50  0000 C CNN
-F 2 "SpeakON:NL4MP-M3" H 3100 3050 50  0001 C CNN
+F 2 "SpeakON:NL4MP-M3_double_left" H 3100 3050 50  0001 C CNN
 F 3 "http://www.neutrik.com/en/speakon/" H 3100 3050 50  0001 C CNN
 	1    3100 3050
